File: Schematics/Electronics/Automatic_sampler.kicad_sch (KiCad schematic)
At the start: 32 parts, among them J1 Sensor, J2 MOTOR_X_CONN, J3 MOTOR_Y_CONN, J4 MOTOR_Z_CONN, J5 Jack-DC, SW1 Final_X, SW2 Final_Y, SW3 Final_Z, SW4 Button, U1 DRV8825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

Commit message: Added end to motor object
Parts:
- removed U10: AZ1117-3.3, symbol Regulator_Linear:AZ1117-3.3
- removed U6: ~, symbol ATSS_Library:TMUX1247
- added U11: ~, Package_TO_SOT_SMD:Texas_R-PDSO-G6, symbol ATSS_Library:TMUX1247
- D1, D2, D3: footprint (none) -> LED_THT:LED_D5.0mm
- J1: footprint (none) -> Connector_PinHeader_2.54mm:PinHeader_1x07_P2.54mm_Vertical
- J2, J3, J4: footprint (none) -> Connector_PinHeader_2.54mm:PinHeader_1x04_P2.54mm_Vertical
- R1, R10, R2, R3, R7, R8, R9: footprint (none) -> Resistor_THT:R_Axial_DIN0204_L3.6mm_D1.6mm_P7.62mm_Horizontal
- RV1: footprint (none) -> Potentiometer_THT:Potentiometer_ACP_CA9-V10_Vertical
- SW1, SW2, SW3, SW4: footprint (none) -> Connector_PinHeader_2.54mm:PinHeader_1x02_P2.54mm_Vertical
Connections:
- net +3.3V: now also U4.36 (3V3), U11. (SEL)
- net +5V: now also U4.39 (VSYS), U11. (SEL)
- net GND: no longer U4.42 (GND)
- net SELV: now also U11. (SEL)
- net at J1.1 (Pin_1): now also U11. (SEL)
- no-connect marks 22 -> 33
Other:
- moved on the sheet: D1, D2, D3, J2, J3, J4, R1, R2, R3, U1, U2, U3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

Commit message: Added KiCad subprojects
Connections:
- net +12V: now also U1.8 (Vmot), U2.8 (Vmot), U3.8 (Vmot); no longer U1. (Vmot), U2. (Vmot), U3. (Vmot)
- net +5V: now also U1.11 (SLEEP), U1.12 (RESET), U2.11 (SLEEP), U2.12 (RESET), U3.11 (SLEEP), U3.12 (RESET); no longer U1. (Vmot), U2. (Vmot), U3. (Vmot)
- net GND: now also U1.1 (GND), U1.7 (GND), U2.1 (GND), U2.7 (GND), U3.1 (GND), U3.7 (GND); no longer U1. (Vmot), U2. (Vmot), U3. (Vmot)
- net MOT_DIR: now also U1.9 (DIR), U2.9 (DIR), U3.9 (DIR); no longer U1. (Vmot), U2. (Vmot), U3. (Vmot)
- net MOT_EN_X: now also U1.16 (ENABLE); no longer U3. (Vmot)
- net MOT_EN_Y: now also U2.16 (ENABLE); no longer U2. (Vmot)
- net MOT_EN_Z: now also U3.16 (ENABLE); no longer U1. (Vmot)
- net MOT_ST: now also U1.10 (STEP), U2.10 (STEP), U3.10 (STEP); no longer U1. (Vmot), U2. (Vmot), U3. (Vmot)
- net at D3.1 (K): now also U3.2 (FAULT); no longer U1. (Vmot)
- net at J4.1 (Pin_1): now also U3.4 (OUT1A); no longer U1. (Vmot)
- net at J4.2 (Pin_2): now also U3.5 (OUT1B); no longer U1. (Vmot)
- net at J4.3 (Pin_3): now also U3.3 (OUT2A); no longer U1. (Vmot)
- net at J4.4 (Pin_4): now also U3.6 (OUT2B); no longer U1. (Vmot)
- net at D2.1 (K): now also U2.2 (FAULT); no longer U2. (Vmot)
- net at D1.1 (K): now also U1.2 (FAULT); no longer U3. (Vmot)
- net at J2.1 (Pin_1): now also U1.4 (OUT1A); no longer U3. (Vmot)
- net at J2.2 (Pin_2): now also U1.5 (OUT1B); no longer U3. (Vmot)
- net at J2.3 (Pin_3): now also U1.3 (OUT2A); no longer U3. (Vmot)
- net at J2.4 (Pin_4): now also U1.6 (OUT2B); no longer U3. (Vmot)
- net at J3.1 (Pin_1): now also U2.4 (OUT1A); no longer U2. (Vmot)
- net at J3.2 (Pin_2): now also U2.5 (OUT1B); no longer U2. (Vmot)
- net at J3.3 (Pin_3): now also U2.3 (OUT2A); no longer U2. (Vmot)
- net at J3.4 (Pin_4): now also U2.6 (OUT2B); no longer U2. (Vmot)
