File: Schematics/Electronics/Automatic_sampler_logic/Automatic_sampler_logic.kicad_pcb (KiCad board)
At the start: 2 copper layers, 15 parts, among them J1 MOT_X_SOCK, J2 MOT_Y_SOCK, J3 MOT_Z_SOCK, J4 Power, J5 FINAL_SOCK, J6 LCD_SOCK, J7 POWER_SOCK, J8 BUTTON_SOCK, J9 MOT_X_SOCK2, U4 Pico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

Commit message: Gerber generated
Parts:
- moved J4 63.4 mm to (122.7, 54.9)
- moved J7 60.7 mm to (150.6, 54.9)
- moved J2 59.0 mm to (110.7, 100.5)
- moved J3 58.7 mm to (110.5, 75.5)
- moved J9 58.2 mm to (112.2, 125.8)
- moved J1 58.1 mm to (105.5, 125.8)
- moved U5 57.5 mm to (133.9, 54.7), turned to 0 degrees
- moved A1 57.3 mm to (152.3, 118.7)
- moved A3 57.3 mm to (118.4, 87.8)
- moved A4 57.3 mm to (118.4, 62.8)
- moved J6 57.3 mm to (139.2, 69.8)
- moved U4 57.3 mm to (157.5, 86.4)
- moved A2 57.0 mm to (118.2, 113.0)
- moved J8 55.0 mm to (175.4, 82.7)
- moved J5 54.9 mm to (175.4, 110.5)
Routing:
- net +5V: track 0.00 -> 145.5 mm
- net +12V: track 0.00 -> 98.7 mm
- net MOT_ST: track 0.00 -> 87.4 mm
- net +3.3V: track 0.00 -> 82.4 mm
- net MOT_DIR: track 0.00 -> 74.6 mm
- net MOT_EN_X: track 0.00 -> 69.9 mm
- net LCD_RS: track 0.00 -> 68.1 mm
- net LCD_E: track 0.00 -> 64.3 mm
- net MOT_EN_Y: track 0.00 -> 51.1 mm
- net SD_MISO: track 0.00 -> 43.2 mm
- net SD_CLK: track 0.00 -> 27.5 mm
- net F_Z: track 0.00 -> 23.3 mm
- net MOT_EN_Z: track 0.00 -> 21.5 mm
- net GND: track 0.00 -> 18.9 mm
- net SD_CS: track 0.00 -> 18.8 mm
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- added copper zone on F.Cu, net GND

Commit message: Added drill files
Other:
- board outline added: 75.1 x 87.6 mm
Changed lines of the file:
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@@
   (gr_rect (start 102.95 48.91) (end 177.95 136.41)
     (stroke (width 0.2) (type default)) (fill none) (layer "F.Cu"))
+  (gr_rect (start 102.9 48.9) (end 178 136.5)
+    (stroke (width 0.1) (type default)) (fill none) (layer "Edge.Cuts"))
   (segment (start 165.162919 72.447081) (end 163.95 73.66) (width 0.25) (layer "F.Cu") (net 1))
   (segment (start 165.162919 72.41) (end 162.2 69.447081) (width 0.25) (layer "F.Cu") (net 1))

Commit message: Updating schematic
Parts:
- removed A1: SD_Card_Module, Arduino_Peripherals:SD_Card_Module
- removed A2, A3, A4: Pololu_Breakout_DRV8825, Module:Pololu_Breakout-16_15.2x20.3mm
- removed J1: MOT_X_SOCK, Connector_PinSocket_2.54mm:PinSocket_1x05_P2.54mm_Vertical
- removed J2: MOT_Y_SOCK, Connector_PinSocket_2.54mm:PinSocket_1x05_P2.54mm_Vertical
- removed J3: MOT_Z_SOCK, Connector_PinSocket_2.54mm:PinSocket_1x05_P2.54mm_Vertical
- removed J4: Power, Connector_PinSocket_2.54mm:PinSocket_1x02_P2.54mm_Vertical
- removed J5: FINAL_SOCK, Connector_PinSocket_2.54mm:PinSocket_1x03_P2.54mm_Vertical
- removed J6: LCD_SOCK, Connector_PinSocket_2.54mm:PinSocket_1x06_P2.54mm_Vertical
- removed J7: POWER_SOCK, Connector_PinSocket_2.54mm:PinSocket_1x03_P2.54mm_Vertical
- removed J8: BUTTON_SOCK, Connector_PinSocket_2.54mm:PinSocket_1x01_P2.54mm_Vertical
- removed J9: MOT_X_SOCK2, Connector_PinSocket_2.54mm:PinSocket_1x05_P2.54mm_Vertical
- removed U4: Pico, MCU_RaspberryPi_and_Boards:RPi_Pico_SMD_TH
- removed U5: LM7805_TO220, Package_TO_SOT_THT:TO-220-3_Vertical
Routing:
- net +5V: track 145.5 -> 0.00 mm
- net +12V: track 98.7 -> 0.00 mm
- net MOT_ST: track 87.4 -> 0.00 mm
- net +3.3V: track 82.4 -> 0.00 mm
- net MOT_DIR: track 74.6 -> 0.00 mm
- net MOT_EN_X: track 69.9 -> 0.00 mm
- net LCD_RS: track 68.1 -> 0.00 mm
- net LCD_E: track 64.3 -> 0.00 mm
- net MOT_EN_Y: track 51.1 -> 0.00 mm
- net SD_MISO: track 43.2 -> 0.00 mm
- net SD_CLK: track 27.5 -> 0.00 mm
- net F_Z: track 23.3 -> 0.00 mm
- net MOT_EN_Z: track 21.5 -> 0.00 mm
- net GND: track 18.9 -> 0.00 mm
- net SD_CS: track 18.8 -> 0.00 mm
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- removed copper zone on F.Cu, net GND
Other:
- board outline removed

Commit message: Made PCB for AS
Parts:
- added A1: Pololu_Breakout_DRV8825, Module:Pololu_Breakout-16_15.2x20.3mm, F.Cu at (130.6, 127.6)
- added A2: Pololu_Breakout_DRV8825, Module:Pololu_Breakout-16_15.2x20.3mm, F.Cu at (157.4, 127.6)
- added A3: Pololu_Breakout_DRV8825, Module:Pololu_Breakout-16_15.2x20.3mm, F.Cu at (183.4, 127.5)
- added A4: Pololu_Breakout_DRV8825, Module:Pololu_Breakout-16_15.2x20.3mm, F.Cu at (209.9, 127.3)
- added C1: 0.33u, Capacitor_THT:C_Disc_D6.0mm_W2.5mm_P5.00mm, F.Cu at (203.0, 90.0)
- added C2: 0.1u, Capacitor_THT:C_Disc_D6.0mm_W2.5mm_P5.00mm, F.Cu at (219.7, 90.0)
- added D1: LED, LED_THT:LED_D5.0mm, F.Cu at (223.5, 102.9)
- added J1: MOT_X_SOCK_2, Connector_JST:JST_PH_B4B-PH-K_1x04_P2.00mm_Vertical, F.Cu at (136.2, 137.2)
- added J2: MOT_X_SOCK_1, Connector_JST:JST_PH_B4B-PH-K_1x04_P2.00mm_Vertical, F.Cu at (162.8, 137.8)
- added J3: MOT_Y_SOCK, Connector_JST:JST_PH_B4B-PH-K_1x04_P2.00mm_Vertical, F.Cu at (189.0, 137.5)
- added J4: Power, Connector_PinSocket_2.54mm:PinSocket_1x02_P2.54mm_Vertical, F.Cu at (189.8, 83.5)
- added J5: FinalSock, Connector_PinSocket_2.54mm:PinSocket_1x04_P2.54mm_Vertical, F.Cu at (185.8, 73.0)
- added J6: MOT_Z_SOCK, Connector_JST:JST_PH_B4B-PH-K_1x04_P2.00mm_Vertical, F.Cu at (215.5, 137.2)
- added R1: 1k, Resistor_THT:R_Axial_DIN0207_L6.3mm_D2.5mm_P7.62mm_Horizontal, F.Cu at (225.8, 90.1)
- added U4: Pico, MCU_RaspberryPi_and_Boards:RPi_Pico_SMD_TH, F.Cu at (159.1, 91.4)
- added U5: LM7805_TO220, Package_TO_SOT_THT:TO-220-3_Vertical, F.Cu at (208.7, 98.2)
Routing:
- net +5V: track 0.00 -> 256.6 mm
- net +12V: track 0.00 -> 232.9 mm
- net FLT: track 0.00 -> 206.8 mm
- net MOT_DIR: track 0.00 -> 125.7 mm
- net MOT_ST: track 0.00 -> 112.5 mm
- net MOT_EN_Z: track 0.00 -> 81.4 mm
- net MOT_EN_Y: track 0.00 -> 52.6 mm
- net MOT_EN_X: track 0.00 -> 42.4 mm
- net F_Z: track 0.00 -> 20.8 mm
- net Net-(A2-B2): track 0.00 -> 10.7 mm
- net Net-(A2-B1): track 0.00 -> 10.5 mm
- net Net-(A3-B2): track 0.00 -> 10.4 mm
- net Net-(A4-B2): track 0.00 -> 10.3 mm
- net Net-(A2-A2): track 0.00 -> 10.3 mm
- net Net-(A2-A1): track 0.00 -> 10.3 mm
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- added copper zone on F.Cu, net GND
